File: hardware/audible.sch (EAGLE design)
At the start: 27 parts, among them IC1 LTC1966CMS8, J1 SQUALL_HEADER, J5 TC2030-JLINK-NL, Q1 FK3503010L, U1 MAX417ESA+, U2 MAX417ESA+

Commit message: Fixed ref names
Parts:
- C1: value 1uF -> 0.01uF
- C10: value 0.1uF -> 22uF
- C2: value 1uF -> 100n
- C3: value 1uF -> 0.1uF
- C4: value 100n -> 0.1uF
- C5: value 1u -> 0.1uF
- C6: value 22uF -> 1u
- C7: value 0.01uF -> 1uF
- C8, C9: value 0.1uF -> 1uF
- R1: value 14k -> 1k
- R3: value 47k -> 10k
- R4: value 14k -> 10k
- R5: value 1k -> 10k
- R6: value 20k -> 14k
- R7: value 10k -> 14k
- R8: value 10k -> 20k
- R9: value 10k -> 47k
- renumbered U$2 to U4, U$3 to U3
Connections:
- net A7: now also R4.1, R5.2; no longer R7.2, R9.1
- net GND: now also C1.1, C3.1, C4.2, C9.2, R3.2, R4.2; no longer C1.2, C2.2, C7.1, C9.1, R8.2, R9.2
- net MIC: now also C7.1; no longer C3.1
- net MIC_AMP_1: now also R6.2; no longer R1.2
- net MIC_AMP_2: now also C2.1, R7.1; no longer C4.1, R4.1
- net N$1: now also C7.2, R9.2; no longer C3.2, R3.2
- net N$10: now also C10.2, R5.1, R8.2; no longer C6.2, R6.2, R7.1
- net N$2: now also C2.2; no longer C4.2
- net N$3: now also C6.2; no longer C5.2
- net N$4: now also R1.2, R6.1; no longer R1.1, R2.2
- net N$5: now also R2.1, R7.2; no longer R4.2, R5.1
- net N$6: now also R3.1; no longer R8.1
- net RMS_BUF: now also R8.1; no longer R6.1
- net VCC: now also C1.2, C3.2, C5.2, C8.1; no longer C10.2, C2.1, C7.2, C9.2
- net VREF: now also C4.1, C9.1, R1.1, R2.2, R9.1; no longer C1.1, C8.1, R2.1, R3.1, R5.2
Other:
- moved on the sheet: C1, C10, C2, C3, C4, C5, C6, C7, C8, C9, R1, R2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
